Commit message: Add Gazebo launch and update robot description

File: src/line_follower_description/urdf/robot.urdf.xacro (robot description, xacro)
@@ -2,74 +2,29 @@
 <robot name="line_follower_robot"
        xmlns:xacro="http://www.ros.org/wiki/xacro">
-  <!-- Include other Xacro files -->
   <xacro:include filename="$(find line_follower_description)/urdf/materials.xacro"/>
   <xacro:include filename="$(find line_follower_description)/urdf/base.xacro"/>
-  <!-- ================= LEFT WHEEL ================= -->
-  <link name="left_wheel">
-    <visual>
-      <origin xyz="0 0 0" rpy="1.5708 0 0"/>
-      <geometry>
-        <cylinder radius="0.05" length="0.03"/>
-      </geometry>
-      <material name="black"/>
-    </visual>
-    <collision>
-      <origin xyz="0 0 0" rpy="1.5708 0 0"/>
-      <geometry>
-        <cylinder radius="0.05" length="0.03"/>
-      </geometry>
-    </collision>
-    <inertial>
-      <mass value="0.3"/>
-      <origin xyz="0 0 0"/>
-      <inertia
-        ixx="0.001"
-        iyy="0.001"
-        izz="0.001"
-        ixy="0"
-        ixz="0"
-        iyz="0"/>
-    </inertial>
-  </link>
-  <!-- ================= RIGHT WHEEL ================= -->
-  <link name="right_wheel">
-    <visual>
-      <origin xyz="0 0 0" rpy="1.5708 0 0"/>
-      <geometry>
-        <cylinder radius="0.05" length="0.03"/>
-      </geometry>
-      <material name="black"/>
-    </visual>
-    <collision>
-      <origin xyz="0 0 0" rpy="1.5708 0 0"/>
-      <geometry>
-        <cylinder radius="0.05" length="0.03"/>
-      </geometry>
-    </collision>
-    <inertial>
-      <mass value="0.3"/>
-      <origin xyz="0 0 0"/>
-      <inertia
-        ixx="0.001"
-        iyy="0.001"
-        izz="0.001"
-        ixy="0"
-        ixz="0"
-        iyz="0"/>
-    </inertial>
-  </link>
-  <!-- ================= LEFT WHEEL JOINT ================= -->
-  <joint name="left_wheel_joint" type="continuous">
-    <parent link="base_link"/>
-    <child link="left_wheel"/>
-    <origin xyz="0 0.11 -0.025" rpy="0 0 0"/>
-    <axis xyz="0 1 0"/>
-  </joint>
-  <!-- ================= RIGHT WHEEL JOINT ================= -->
-  <joint name="right_wheel_joint" type="continuous">
-    <parent link="base_link"/>
-    <child link="right_wheel"/>
-    <origin xyz="0 -0.11 -0.025" rpy="0 0 0"/>
-    <axis xyz="0 1 0"/>
-  </joint>
+  <xacro:include filename="$(find line_follower_description)/urdf/wheels.xacro"/>
+  <xacro:wheel prefix="left" y_position="0.11"/>
+  <xacro:wheel prefix="right" y_position="-0.11"/>
+    <!-- Gazebo Differential Drive Plugin -->
+  <gazebo>
+    <plugin
+      filename="libgazebo_ros_diff_drive.so"
+      name="diff_drive_controller">
+      <ros>
+        <namespace>/</namespace>
+      </ros>
+      <update_rate>50</update_rate>
+      <left_joint>left_wheel_joint</left_joint>
+      <right_joint>right_wheel_joint</right_joint>
+      <wheel_separation>0.22</wheel_separation>
+      <wheel_diameter>0.10</wheel_diameter>
+      <command_topic>cmd_vel</command_topic>
+      <odometry_topic>odom</odometry_topic>
+      <odometry_frame>odom</odometry_frame>
+      <robot_base_frame>base_link</robot_base_frame>
+      <publish_odom>true</publish_odom>
+      <publish_tf>true</publish_tf>
+    </plugin>
+  </gazebo>
 </robot>
